Commit message: fix(cart_urdf): cart_with_arm.urdf.xacro — добавить отсутствующие xacro:arg (enable_camera_realsense, enable_extra_floor_tofs, enable_camera_oak/orbbec, enable_pace_battery) и property robot_model
Причина падения 'ros2 launch cart_xarm_bringup cart_xarm6_gz.launch.py':
- cart-base.urdf.xacro использует $(arg enable_camera_realsense) и др.,
  которые объявлены только в cart.urdf.xacro; наш файл-обёртка их не объявлял
  -> xacro: 'Undefined substitution argument enable_camera_realsense'
- cart-base.urdf.xacro также использует ${robot_model.startswith('c2w')}
  (property из cart.urdf.xacro) -> после фикса аргументов упало бы
  'name robot_model is not defined'. Добавлен <xacro:property name="robot_model" .../>

Проверено локально: xacro генерирует валидный URDF (54 link, arm_mount_joint
base_link->arm_mount_link xyz=-0.0075 0 0.849, вакуумный гриппер + camera_link).

File: src/r2_robot/quasi_cart_description/urdf/cart_with_arm.urdf.xacro (robot description, xacro)
@@ -20,4 +20,9 @@
     <xacro:arg name="camera_roll_offset" default="0.0"/>
     <xacro:arg name="camera_pitch_offset" default="0.0"/>
+    <xacro:arg name="enable_extra_floor_tofs" default="false"/>
+    <xacro:arg name="enable_camera_realsense" default="false"/>
+    <xacro:arg name="enable_camera_oak" default="false"/>
+    <xacro:arg name="enable_camera_orbbec" default="false"/>
+    <xacro:arg name="enable_pace_battery" default="true"/>
     <!-- Аргументы руки (пробрасываются в cart-arm.xacro) -->
     <xacro:arg name="arm_dof" default="6"/>
@@ -28,4 +33,9 @@
     <xacro:arg name="arm_ros2_control_plugin" default="gz_ros2_control/GazeboSimSystem"/>
     <xacro:property name="var_simulator" value="$(arg simulator)"/>
+    <!-- property robot_model ОБЯЗАТЕЛЕН: cart-base.urdf.xacro использует
+         выражение ${robot_model.startswith('c2w')} (есть в cart.urdf.xacro,
+         но не в этом файле-обёртке — без него xacro падает с
+         "name 'robot_model' is not defined") -->
+    <xacro:property name="robot_model" value="$(arg robot_model)"/>
     <xacro:property name="drive" value="differential"/>
     <material name="white_pva"><color rgba="1 1 1 1"/></material>
