Commit message: feat(sim): начальная поза руки, MoveIt без ручного use_sim_time, TF колёс, RViz-запуск, документация
Тележка (cart_xarm_bringup):
- начальная поза руки через initial_value gz_ros2_control (аргумент
  arm_initial_positions, по умолчанию рука вбок над платформой)
- MoveIt: use_sim_time передаётся в _robot_moveit_common явно (его
  default False перекрывал SetParameter — отсюда ручной param set);
  фиксер удалён; static TF world->link_base отключён (publish_attach_tf),
  вместо него link_base->world — без двух родителей у link_base;
  старт MoveIt отложен на 12 с
- колёса: JointStatePublisher в Gazebo + мост /cart/wheel_joint_states,
  joint_state_publisher сливает с /joint_states для robot_state_publisher
  (раньше drive_wheel_* без TF)
- мосты /cmd_vel и /odom; убран дублирующий мост /joint_states
- новый cart_xarm6_rviz.launch.py: только RViz + ползунки суставов

Рука отдельно (xarm_gz_bringup):
- table_gz.world: блок встроен (model://cylinder_block не находился,
  gz sim завершался)
- спавн на верх столешницы (z=1.015) и начальная поза с гриппером над
  столом (в нулевой позе присоска уходила в стол -> PATH_TOLERANCE_VIOLATED)
- use_sim_time для MoveIt без фиксера

xarm_grasping: Marker.lifetime через to_msg(), float в полях маркеров
(abort процесса в rosidl-конвертере).

README.md: установка с нуля, сборка, все сценарии запуска, проверка,
use_sim_time, типичные проблемы. INSTALL_RUN.md -> ссылка на README.

Co-Authored-By: Claude Opus 5.5 <noreply@anthropic.com>

File: src/r2_robot/quasi_cart_description/urdf/cart_with_arm.urdf.xacro (robot description, xacro)
@@ -83,4 +83,18 @@
             -->
             <xacro:include filename="cart-sensors.ign.xacro" />
+            <!-- Состояние ведущих колёс: их не публикует ни ros2_control
+                 (joint_state_broadcaster знает только суставы руки), ни что-то
+                 ещё -> у drive_wheel_*_link не было TF ("No transform" в RViz).
+                 Gazebo публикует реальные углы колёс, gz_bridge отдаёт их в
+                 /cart/wheel_joint_states, joint_state_publisher в launch
+                 сливает их с /joint_states руки для robot_state_publisher. -->
+            <gazebo>
+              <plugin filename="gz-sim-joint-state-publisher-system"
+                      name="gz::sim::systems::JointStatePublisher">
+                <topic>/model/cart/wheel_joint_states</topic>
+                <joint_name>drive_wheel_left_joint</joint_name>
+                <joint_name>drive_wheel_right_joint</joint_name>
+              </plugin>
+            </gazebo>
         </xacro:if>
     </xacro:if>

File: src/xarm_ros2/xarm_description/urdf/xarm6/xarm6.ros2_control.xacro (robot description, xacro)
@@ -1,4 +1,11 @@
 <?xml version="1.0"?>
 <robot xmlns:xacro="http://ros.org/wiki/xacro">
+  <!-- Начальная поза суставов в симуляции (gz_ros2_control: initial_value).
+       6 чисел через пробел (рад), joint1..joint6; пусто — все нули, как раньше.
+       Реальное железо (UFRobotSystemHardware) этот параметр игнорирует.
+       Первое объявление xacro:arg побеждает: родительский xacro может задать
+       свой default до include. -->
+  <xacro:arg name="xarm_initial_positions" default=""/>
+  <xacro:property name="xarm_init_pos" value="$(arg xarm_initial_positions)"/>
   <xacro:macro name="xarm6_ros2_control" params="prefix
     velocity_control:='false'
@@ -44,5 +51,9 @@
           <param name="max">3.14</param>
         </command_interface>
-        <state_interface name="position"/>
+        <state_interface name="position">
+          <xacro:if value="${xarm_init_pos != ''}">
+            <param name="initial_value">${float(xarm_init_pos.split()[0])}</param>
+          </xacro:if>
+        </state_interface>
         <state_interface name="velocity"/>
         <!-- <state_interface name="effort"/> -->
@@ -57,5 +68,9 @@
           <param name="max">3.14</param>
         </command_interface>
-        <state_interface name="position"/>
+        <state_interface name="position">
+          <xacro:if value="${xarm_init_pos != ''}">
+            <param name="initial_value">${float(xarm_init_pos.split()[1])}</param>
+          </xacro:if>
+        </state_interface>
         <state_interface name="velocity"/>
         <!-- <state_interface name="effort"/> -->
@@ -70,5 +85,9 @@
           <param name="max">3.14</param>
         </command_interface>
-        <state_interface name="position"/>
+        <state_interface name="position">
+          <xacro:if value="${xarm_init_pos != ''}">
+            <param name="initial_value">${float(xarm_init_pos.split()[2])}</param>
+          </xacro:if>
+        </state_interface>
         <state_interface name="velocity"/>
         <!-- <state_interface name="effort"/> -->
@@ -83,5 +102,9 @@
           <param name="max">3.14</param>
         </command_interface>
-        <state_interface name="position"/>
+        <state_interface name="position">
+          <xacro:if value="${xarm_init_pos != ''}">
+            <param name="initial_value">${float(xarm_init_pos.split()[3])}</param>
+          </xacro:if>
+        </state_interface>
         <state_interface name="velocity"/>
         <!-- <state_interface name="effort"/> -->
@@ -96,5 +119,9 @@
           <param name="max">3.14</param>
         </command_interface>
-        <state_interface name="position"/>
+        <state_interface name="position">
+          <xacro:if value="${xarm_init_pos != ''}">
+            <param name="initial_value">${float(xarm_init_pos.split()[4])}</param>
+          </xacro:if>
+        </state_interface>
         <state_interface name="velocity"/>
         <!-- <state_interface name="effort"/> -->
@@ -109,5 +136,9 @@
           <param name="max">3.14</param>
         </command_interface>
-        <state_interface name="position"/>
+        <state_interface name="position">
+          <xacro:if value="${xarm_init_pos != ''}">
+            <param name="initial_value">${float(xarm_init_pos.split()[5])}</param>
+          </xacro:if>
+        </state_interface>
         <state_interface name="velocity"/>
         <!-- <state_interface name="effort"/> -->
