Commit message: add c2l scalling

File: src/r2_robot/quasi_cart_description/urdf/c2l-v3.urdf.xacro (robot description, xacro)
@@ -2,4 +2,13 @@
 <robot name="quasi_c2l-v3" xmlns:xacro="http://ros.org/wiki/xacro">
   <xacro:property name="cart_version" value="v3" />
+  <!-- Меш корпуса: default — только если не задан раньше
+       (c2l-v3-scaled.urdf.xacro подставляет масштабированный меш c2) -->
+  <xacro:property name="base_mesh" default="base_link_c2l-v3.stl" />
+  <xacro:property name="base_mesh_scale" default="1 1 1" />
+  <!-- Крепление руки (cart-arm.xacro), base_link: по CAD (C2R.000.000.000)
+       база руки смещена на 250 мм от центра к ручке (-X) и на 129.5 мм
+       к левому краю, если стоять у ручки лицом вперёд (+Y);
+       z — верх крыши, та же высота, что у c2 -->
+  <xacro:property name="arm_mount_xyz" default="-0.25 0.1295 0.849" />
   <link name="base_link">
     <inertial>
@@ -12,5 +21,6 @@
       <origin xyz="0 0 0" rpy="0 0 0" />
       <geometry>
-        <mesh filename="file://$(find quasi_cart_description)/meshes/base_link_c2l-v3.stl" />
+        <mesh filename="file://$(find quasi_cart_description)/meshes/${base_mesh}"
+              scale="${base_mesh_scale}" />
       </geometry>
       <material name="">
@@ -21,5 +31,6 @@
       <origin xyz="0 0 0" rpy="0 0 0" />
       <geometry>
-        <mesh filename="file://$(find quasi_cart_description)/meshes/base_link_c2l-v3.stl" />
+        <mesh filename="file://$(find quasi_cart_description)/meshes/${base_mesh}"
+              scale="${base_mesh_scale}" />
       </geometry>
     </collision>

File: src/r2_robot/quasi_cart_description/urdf/cart-arm.xacro (robot description, xacro)
@@ -24,4 +24,9 @@
   <xacro:arg name="arm_ros2_control_plugin" default="gz_ros2_control/GazeboSimSystem"/>
   <!-- ==================== Фланец крепления на крыше тележки ==================== -->
+  <!-- Точка крепления зависит от тележки: файл модели (<robot_model>.urdf.xacro,
+       подключается раньше) может задать свойство arm_mount_xyz.
+       Default — центр платформы c2: x=-0.0075 (середина [-0.359..0.359]),
+       y=0, z=верх 0.849 -->
+  <xacro:property name="arm_mount_xyz" default="-0.0075 0.0 0.849"/>
   <xacro:macro name="arm_mount_link" params="">
     <!-- Фиктивный link-«фланец» на верхней плоской платформе тележки -->
@@ -30,6 +35,5 @@
       <parent link="base_link"/>
       <child link="arm_mount_link"/>
-      <!-- центр платформы: x=-0.0075 (середина [-0.359..0.359]), y=0, z=верх 0.849 -->
-      <origin xyz="-0.0075 0.0 0.849" rpy="0 0 0"/>
+      <origin xyz="${arm_mount_xyz}" rpy="0 0 0"/>
     </joint>
   </xacro:macro>

Commit message: changes arm position testing camera griper

File: src/r2_robot/quasi_cart_description/urdf/c2l-v3.urdf.xacro (robot description, xacro)
@@ -10,5 +10,5 @@
        к левому краю, если стоять у ручки лицом вперёд (+Y);
        z — верх крыши, та же высота, что у c2 -->
-  <xacro:property name="arm_mount_xyz" default="-0.25 0.1295 0.849" />
+  <xacro:property name="arm_mount_xyz" default="-0.25 -0.1295 0.849" />
   <link name="base_link">
     <inertial>

File: src/r2_robot/quasi_cart_description/urdf/cart_with_arm.urdf.xacro (robot description, xacro)
@@ -15,5 +15,5 @@
     <!-- ==================== Аргументы ==================== -->
     <xacro:arg name="use_sim" default="false" />
-    <xacro:arg name="robot_model" default="c2" />
+    <xacro:arg name="robot_model" default="c2l-v3-scaled" />
     <xacro:arg name="simulator" default="ignition" />
     <xacro:arg name="enable_floor_tofs" default="true" />
