Commit message: arm position and navstack

File: src/r2_robot/quasi_cart_description/urdf/c2-v3.urdf.xacro (robot description, xacro)
@@ -282,7 +282,11 @@
       xyz="0 0 0" />
   </joint>
+    <!-- Симуляция (gz DiffDrive): колёса вращаются (continuous, обе оси +y, т.к. DiffDrive применяет
+       один знак скорости к обоим колёсам). В исходной модели c1 — revolute с пределами 0..0 и левой осью -y.
+       sim_wheel_separation — расстояние между ведущими колёсами, м (считано по суставам). -->
+  <xacro:property name="sim_wheel_separation" value="0.354" />
   <joint
     name="drive_wheel_right_joint"
-    type="revolute">
+    type="continuous">
     <origin xyz="0 -0.177 0" rpy="0 0 0"/>
     <parent
@@ -292,13 +296,9 @@
     <axis
       xyz="0 1 0" />
-    <limit
-      lower="0"
-      upper="0"
-      effort="0"
-      velocity="0" />
+    <limit effort="60" velocity="20" />
   </joint>
   <joint
     name="drive_wheel_left_joint"
-    type="revolute">
+    type="continuous">
     <origin xyz="0 0.177 0" rpy="0 0 0"/>
     <parent
@@ -307,10 +307,6 @@
       link="drive_wheel_left_link" />
     <axis
-      xyz="0 -1 0" />
-    <limit
-      lower="0"
-      upper="0"
-      effort="0"
-      velocity="0" />
+      xyz="0 1 0" />
+    <limit effort="60" velocity="20" />
   </joint>
   <joint

File: src/r2_robot/quasi_cart_description/urdf/c2l-v3.urdf.xacro (robot description, xacro)
@@ -276,7 +276,11 @@
     <axis xyz="0 0 0" />
   </joint>
+    <!-- Симуляция (gz DiffDrive): колёса вращаются (continuous, обе оси +y, т.к. DiffDrive применяет
+       один знак скорости к обоим колёсам). В исходной модели c1 — revolute с пределами 0..0 и левой осью -y.
+       sim_wheel_separation — расстояние между ведущими колёсами, м (считано по суставам). -->
+  <xacro:property name="sim_wheel_separation" value="0.50386" />
   <joint
     name="drive_wheel_right_joint"
-    type="revolute">
+    type="continuous">
     <origin
       xyz="0 -0.25193 0"
@@ -288,13 +292,9 @@
     <axis
       xyz="0 1 0" />
-    <limit
-      lower="0"
-      upper="0"
-      effort="0"
-      velocity="0" />
+    <limit effort="60" velocity="20" />
   </joint>
   <joint
     name="drive_wheel_left_joint"
-    type="revolute">
+    type="continuous">
     <origin
       xyz="0 0.25193 0"
@@ -305,10 +305,6 @@
       link="drive_wheel_left_link" />
     <axis
-      xyz="0 -1 0" />
-    <limit
-      lower="0"
-      upper="0"
-      effort="0"
-      velocity="0" />
+      xyz="0 1 0" />
+    <limit effort="60" velocity="20" />
   </joint>
   <joint

File: src/r2_robot/quasi_cart_description/urdf/c2m-v3.urdf.xacro (robot description, xacro)
@@ -246,7 +246,11 @@
       xyz="0 0 0" />
   </joint>
+    <!-- Симуляция (gz DiffDrive): колёса вращаются (continuous, обе оси +y, т.к. DiffDrive применяет
+       один знак скорости к обоим колёсам). В исходной модели c1 — revolute с пределами 0..0 и левой осью -y.
+       sim_wheel_separation — расстояние между ведущими колёсами, м (считано по суставам). -->
+  <xacro:property name="sim_wheel_separation" value="0.354" />
   <joint
     name="drive_wheel_right_joint"
-    type="revolute">
+    type="continuous">
     <origin xyz="0 -0.177 0" rpy="0 0 0"/>
     <parent
@@ -256,13 +260,9 @@
     <axis
       xyz="0 1 0" />
-    <limit
-      lower="0"
-      upper="0"
-      effort="0"
-      velocity="0" />
+    <limit effort="60" velocity="20" />
   </joint>
   <joint
     name="drive_wheel_left_joint"
-    type="revolute">
+    type="continuous">
     <origin xyz="0 0.177 0" rpy="0 0 0"/>
     <parent
@@ -271,10 +271,6 @@
       link="drive_wheel_left_link" />
     <axis
-      xyz="0 -1 0" />
-    <limit
-      lower="0"
-      upper="0"
-      effort="0"
-      velocity="0" />
+      xyz="0 1 0" />
+    <limit effort="60" velocity="20" />
   </joint>
   <joint

File: src/r2_robot/quasi_cart_description/urdf/c2t-v3.urdf.xacro (robot description, xacro)
@@ -267,7 +267,11 @@
     <axis xyz="0 0 0" />
   </joint>
+    <!-- Симуляция (gz DiffDrive): колёса вращаются (continuous, обе оси +y, т.к. DiffDrive применяет
+       один знак скорости к обоим колёсам). В исходной модели c1 — revolute с пределами 0..0 и левой осью -y.
+       sim_wheel_separation — расстояние между ведущими колёсами, м (считано по суставам). -->
+  <xacro:property name="sim_wheel_separation" value="0.50386" />
   <joint
     name="drive_wheel_right_joint"
-    type="revolute">
+    type="continuous">
     <origin
       xyz="0 -0.25193 0"
@@ -279,13 +283,9 @@
     <axis
       xyz="0 1 0" />
-    <limit
-      lower="0"
-      upper="0"
-      effort="0"
-      velocity="0" />
+    <limit effort="60" velocity="20" />
   </joint>
   <joint
     name="drive_wheel_left_joint"
-    type="revolute">
+    type="continuous">
     <origin
       xyz="0 0.25193 0"
@@ -296,10 +296,6 @@
       link="drive_wheel_left_link" />
     <axis
-      xyz="0 -1 0" />
-    <limit
-      lower="0"
-      upper="0"
-      effort="0"
-      velocity="0" />
+      xyz="0 1 0" />
+    <limit effort="60" velocity="20" />
   </joint>
   <joint

File: src/r2_robot/quasi_cart_description/urdf/c2w-v3.urdf.xacro (robot description, xacro)
@@ -236,7 +236,11 @@
     <axis xyz="0 0 0" />
   </joint>
+    <!-- Симуляция (gz DiffDrive): колёса вращаются (continuous, обе оси +y, т.к. DiffDrive применяет
+       один знак скорости к обоим колёсам). В исходной модели c1 — revolute с пределами 0..0 и левой осью -y.
+       sim_wheel_separation — расстояние между ведущими колёсами, м (считано по суставам). -->
+  <xacro:property name="sim_wheel_separation" value="0.50386" />
   <joint
     name="drive_wheel_right_joint"
-    type="revolute">
+    type="continuous">
     <origin
       xyz="0 -0.25193 0"
@@ -248,13 +252,9 @@
     <axis
       xyz="0 1 0" />
-    <limit
-      lower="0"
-      upper="0"
-      effort="0"
-      velocity="0" />
+    <limit effort="60" velocity="20" />
   </joint>
   <joint
     name="drive_wheel_left_joint"
-    type="revolute">
+    type="continuous">
     <origin
       xyz="0 0.25193 0"
@@ -265,10 +265,6 @@
       link="drive_wheel_left_link" />
     <axis
-      xyz="0 -1 0" />
-    <limit
-      lower="0"
-      upper="0"
-      effort="0"
-      velocity="0" />
+      xyz="0 1 0" />
+    <limit effort="60" velocity="20" />
   </joint>
   <joint

File: src/r2_robot/quasi_cart_description/urdf/cart-arm.xacro (robot description, xacro)
@@ -32,4 +32,6 @@
        пробел. Имена = имена моделей в мире, у каждой link «link», модели НЕ static.
        На каждую — свой плагин и топики /vacuum/<модель>/{attach,detach,state}. -->
+  <!-- none — без присоски-сварки (сценарий навигации без нод захвата: иначе pick_box остаётся
+       приваренным к руке с момента загрузки и тележка тащит его за собой) -->
   <xacro:arg name="vacuum_targets" default="pick_box"/>
   <!-- Плагин DetachableJoint на каждую модель из списка (xacro без циклов —
@@ -119,5 +121,5 @@
     -->
     <xacro:if value="$(arg use_sim)">
-      <xacro:vacuum_joints targets="${'$(arg vacuum_targets)'.split()}"/>
+      <xacro:vacuum_joints targets="${[t for t in '$(arg vacuum_targets)'.split() if t != 'none']}"/>
       <gazebo>
         <!-- Поза модели робота в мире (10 Гц) — для проверки касания присоской -->

File: src/r2_robot/quasi_cart_description/urdf/cart-drive-differential.urdf.xacro (robot description, xacro)
@@ -33,11 +33,8 @@
     </visual>
     <collision>
-      <origin
-          xyz="0 0 0"
-          rpy="0 0 0" />
-      <geometry>
-        <mesh
-            filename="file://$(find quasi_cart_description)/meshes/drive_wheel_right_link.STL" />
-      </geometry>
+      <!-- Коллизия колеса в симуляции — цилиндр вместо STL-сетки (у сетки 590..7592 треугольников,
+           контакт «прыгал» и тележка подпрыгивала при езде вперёд). Размеры по пятну контакта сетки. -->
+      <origin xyz="0 0 0" rpy="${pi/2} 0 0" />
+      <geometry><cylinder radius="0.065" length="0.04" /></geometry>
     </collision>
   </link>
@@ -73,11 +70,8 @@
     </visual>
     <collision>
-      <origin
-          xyz="0 0 0"
-          rpy="0 0 0" />
-      <geometry>
-        <mesh
-            filename="file://$(find quasi_cart_description)/meshes/drive_wheel_left_link.STL" />
-      </geometry>
+      <!-- Коллизия колеса в симуляции — цилиндр вместо STL-сетки (у сетки 590..7592 треугольников,
+           контакт «прыгал» и тележка подпрыгивала при езде вперёд). Размеры по пятну контакта сетки. -->
+      <origin xyz="0 0 0" rpy="${pi/2} 0 0" />
+      <geometry><cylinder radius="0.065" length="0.04" /></geometry>
     </collision>
   </link>
@@ -153,11 +147,8 @@
     </visual>
     <collision>
-      <origin
-          xyz="0 0 0"
-          rpy="0 0 0" />
-      <geometry>
-        <mesh
-            filename="file://$(find quasi_cart_description)/meshes/wheel_rr_link.stl" />
-      </geometry>
+      <!-- Коллизия колеса в симуляции — цилиндр вместо STL-сетки (у сетки 590..7592 треугольников,
+           контакт «прыгал» и тележка подпрыгивала при езде вперёд). Размеры по пятну контакта сетки. -->
+      <origin xyz="0 0 0" rpy="${pi/2} 0 0" />
+      <geometry><cylinder radius="0.062" length="0.032" /></geometry>
     </collision>
   </link>
@@ -251,11 +242,8 @@
     </visual>
     <collision>
-      <origin
-          xyz="0 0 0"
-          rpy="0 0 0" />
-      <geometry>
-        <mesh
-            filename="file://$(find quasi_cart_description)/meshes/wheel_rl_link.stl" />
-      </geometry>
+      <!-- Коллизия колеса в симуляции — цилиндр вместо STL-сетки (у сетки 590..7592 треугольников,
+           контакт «прыгал» и тележка подпрыгивала при езде вперёд). Размеры по пятну контакта сетки. -->
+      <origin xyz="0 0 0" rpy="${pi/2} 0 0" />
+      <geometry><cylinder radius="0.062" length="0.032" /></geometry>
     </collision>
   </link>

File: src/r2_robot/quasi_cart_description/urdf/cart-sensors.ign.xacro (robot description, xacro)
@@ -7,11 +7,46 @@
   <!-- false, если Sensors-система уже объявлена в world-файле (см. cart_with_arm) -->
   <xacro:arg name="model_sensors_plugin" default="true"/>
-  <gazebo>
-    <plugin
-            filename="ignition-gazebo-velocity-control-system"
-            name="ignition::gazebo::systems::VelocityControl">
-      <topic>/model/cart/cmd_vel</topic>
-    </plugin>
-  </gazebo>
+  <!-- Привод в симуляции. diff (по умолчанию) — gz DiffDrive: крутит ведущие колёса
+       drive_wheel_*_joint, тележка едет за счёт сцепления колёс с полом (две задние
+       ведущие колеса, два передних кастера). velocity — прежний VelocityControl: задаёт
+       скорость всему корпусу, колёса не вращаются; при длинном заднем ходе тележка
+       с рукой заваливалась (STATUS K10). Выбор: xacro-аргумент sim_drive. -->
+  <xacro:arg name="sim_drive" default="diff"/>
+  <xacro:arg name="sim_wheel_radius" default="0.065"/>
+  <xacro:if value="${'$(arg sim_drive)' == 'diff'}">
+    <gazebo>
+      <plugin filename="gz-sim-diff-drive-system" name="gz::sim::systems::DiffDrive">
+        <topic>/model/cart/cmd_vel</topic>
+        <left_joint>drive_wheel_left_joint</left_joint>
+        <right_joint>drive_wheel_right_joint</right_joint>
+        <wheel_separation>${sim_wheel_separation}</wheel_separation>
+        <wheel_radius>$(arg sim_wheel_radius)</wheel_radius>
+        <!-- пределы, как у Nav2 (nav2_cart.yaml): вперёд 0.4, назад 0.2 м/с; запас по ускорению
+             не даёт колёсам рвануть сильнее, чем держит сцепление -->
+        <max_linear_velocity>1.1</max_linear_velocity>
+        <min_linear_velocity>-0.75</min_linear_velocity>
+        <max_angular_velocity>1.5</max_angular_velocity>
+        <min_angular_velocity>-1.5</min_angular_velocity>
+        <max_linear_acceleration>1.5</max_linear_acceleration>
+        <min_linear_acceleration>-1.5</min_linear_acceleration>
+        <max_angular_acceleration>3.0</max_angular_acceleration>
+        <min_angular_acceleration>-3.0</min_angular_acceleration>
+        <!-- одометрия тележки идёт от OdometryPublisher (ниже, /model/cart/tf);
+             собственную одометрию DiffDrive уводим на другие топики -->
+        <odom_publish_frequency>5</odom_publish_frequency>
+        <odom_topic>/model/cart/diff_odom</odom_topic>
+        <tf_topic>/model/cart/diff_tf</tf_topic>
+      </plugin>
+    </gazebo>
+  </xacro:if>
+  <xacro:unless value="${'$(arg sim_drive)' == 'diff'}">
+    <gazebo>
+      <plugin
+              filename="ignition-gazebo-velocity-control-system"
+              name="ignition::gazebo::systems::VelocityControl">
+        <topic>/model/cart/cmd_vel</topic>
+      </plugin>
+    </gazebo>
+  </xacro:unless>
   <!-- <gazebo>
     <plugin

File: src/r2_robot/quasi_cart_description/urdf/cart_with_arm.urdf.xacro (robot description, xacro)
@@ -89,4 +89,14 @@
             -->
             <xacro:include filename="cart-sensors.ign.xacro" />
+            <!-- Сцепление (DiffDrive): ведущие колёса держатся за пол, кастеры скользят
+                 (иначе тележка не повернёт: кастер с трением 1 тормозит боком).
+                 Кастеры в URDF — fixed-суставы и без preserveFixedJoint склеиваются
+                 с корпусом, трение у склеенных звеньев пропадает. -->
+            <gazebo reference="drive_wheel_left_link"><mu1>1.5</mu1><mu2>1.5</mu2></gazebo>
+            <gazebo reference="drive_wheel_right_link"><mu1>1.5</mu1><mu2>1.5</mu2></gazebo>
+            <gazebo reference="caster_wheel_left_joint"><preserveFixedJoint>true</preserveFixedJoint></gazebo>
+            <gazebo reference="caster_wheel_right_joint"><preserveFixedJoint>true</preserveFixedJoint></gazebo>
+            <gazebo reference="caster_wheel_left_link"><mu1>0.02</mu1><mu2>0.02</mu2></gazebo>
+            <gazebo reference="caster_wheel_right_link"><mu1>0.02</mu1><mu2>0.02</mu2></gazebo>
             <!-- Состояние ведущих колёс: их не публикует ни ros2_control
                  (joint_state_broadcaster знает только суставы руки), ни что-то
