Commit message: add changes

File: src/r2_robot/quasi_camera_description/urdf/gripper_camera.xacro (robot description, xacro)
@@ -19,8 +19,10 @@
               mount_xyz:='0.075 0 0.030' mount_rpy:='${pi} ${-pi/2} 0'
               use_nominal_extrinsics:=true add_gz_sensor:=false preview:=false">
-    <!-- Кронштейн: бокс-заглушка (до появления STL из CAD). Лежит рядом с
-         присоской (x ≥ 0.0375, присоска до x=0.0375), коллизий с ней нет. -->
+    <!-- Кронштейн: бокс-заглушка (до появления STL из CAD). Привязан к mount_xyz:
+         центр на 18.75 мм (полтолщины бокса) ближе к оси, чем винт камеры;
+         при дефолте 0.075 → x=0.05625, рядом с присоской (до x=0.0375). -->
+    <xacro:property name="_m" value="${[float(v) for v in mount_xyz.split()]}"/>
     <joint name="${name}_bracket_joint" type="fixed">
-      <origin xyz="0.05625 0 0.030" rpy="0 0 0"/>
+      <origin xyz="${_m[0] - 0.01875} ${_m[1]} ${_m[2]}" rpy="0 0 0"/>
       <parent link="${parent}"/>
       <child link="${name}_bracket_link"/>

File: src/r2_robot/quasi_cart_description/urdf/cart-arm.xacro (robot description, xacro)
@@ -2,9 +2,11 @@
 <!--
   cart-arm.xacro — интеграция манипулятора xArm6 с вакуумным гриппером
-  и камерой на ЭФ (Realsense D435i) в URDF тележки quasi_cart (r2_robot).
-  Манипулятор ставится СТРОГО ПО ЦЕНТРУ верхней плоской платформы тележки.
-  Координаты верхнего листа base_link (по мешу base_link_c2-v3.stl):
-      z_top = 0.849 м,  x[-0.359 .. 0.359], y[-0.235 .. 0.235]
-  Центр платформы в base_link: (-0.0075, 0.0) — сюда крепится база руки.
+  и камерой на ЭФ (camera_model: gemini335le по умолчанию | d435i) в URDF
+  тележки quasi_cart (r2_robot).
+  Точка крепления базы руки — свойство arm_mount_xyz (в base_link):
+    - модель тележки может задать своё (c2l-v3*: -0.25 -0.1295 0.849, у края);
+    - иначе дефолт ниже — центр крыши c2 (-0.0075 0 0.849), меш
+      base_link_c2-v3.stl: z_top = 0.849 м, x[-0.359 .. 0.359], y[-0.235 .. 0.235].
+  Доп. смещение/поворот — аргументы arm_offset_xyz / arm_offset_rpy.
   Использование (из cart_with_arm.urdf.xacro):
       <xacro:include filename="cart-arm.xacro"/>
@@ -53,8 +55,8 @@
       attach_to="arm_mount_link" — рука ЖЁСТКО вшита в URDF тележки;
       add_vacuum_gripper=true   — вакуумная присоска на link_eef;
-      add_realsense_d435i=true  — камера гриппера: топики camera/color/image_raw,
-                                  camera/color/camera_info, camera/depth/points
-                                  публикуются из Gazebo (realsense_gz при
-                                  ros2_control_plugin=gz_ros2_control/GazeboSimSystem).
+      камера гриппера по camera_model: gemini335le -> add_gripper_camera
+                                  (топики /gripper_camera/..., quasi_camera_description);
+                                  d435i -> add_realsense_d435i (старые /camera/...,
+                                  realsense_gz). gz-сенсор включается при use_sim.
     -->
     <xacro:xarm_device

File: src/r2_robot/quasi_cart_description/urdf/cart_with_arm.urdf.xacro (robot description, xacro)
@@ -3,10 +3,10 @@
   cart_with_arm.urdf.xacro — тележка quasi_cart (репозиторий r2_robot)
   + манипулятор xArm6 с вакуумным гриппером и камерой на ЭФ.
-  Рука расположена ПО ЦЕНТРУ верхней плоской платформы тележки:
-  joint arm_mount_joint (base_link -> arm_mount_link, xyz="-0.0075 0 0.849"),
+  Рука стоит на крыше тележки: joint arm_mount_joint (base_link -> arm_mount_link,
+  xyz = arm_mount_xyz: для c2 центр -0.0075 0 0.849, для c2l-v3* -0.25 -0.1295 0.849),
   затем world_joint руки (arm_mount_link -> link_base).
   Этот URDF имеет ПРЯМУЮ ссылку на добавленный манипулятор:
       <xacro:include filename="cart-arm.xacro"/>
-      <xacro:mount_xarm6_on_cart/>   # xArm6 + add_vacuum_gripper + D435i camera
+      <xacro:mount_xarm6_on_cart/>   # xArm6 + add_vacuum_gripper + камера (camera_model)
   Проверка генерации:
       xacro cart_with_arm.urdf.xacro use_sim:=true
@@ -102,5 +102,5 @@
     <!-- Ссылка на руку: include + вызов макроса mount_xarm6_on_cart.
          Внутри: xArm6 dof=$(arg arm_dof) + add_vacuum_gripper=true
-         + add_realsense_d435i=true (камера гриппера для grasp_analyzer). -->
+         + камера гриппера по camera_model (для grasp_analyzer). -->
     <xacro:include filename="cart-arm.xacro"/>
     <xacro:mount_xarm6_on_cart/>

Commit message: grasp method

File: src/r2_robot/quasi_camera_description/urdf/gripper_camera.xacro (robot description, xacro)
@@ -5,24 +5,31 @@
   (параметры add_gripper_camera / gripper_camera_model / ...).
   Геометрия (в фрейме link_eef, Z — по оси инструмента, присоска до z=0.1265,
-  TCP z=0.126, радиус присоски ~0.046 м):
-    mount_xyz = 0.075 0 0.030   — винт камеры на 75 мм от оси и 30 мм от фланца
-    mount_rpy = π -π/2 0        — ось X камеры (взгляд) = ось Z инструмента;
-                                  проверка: R·[1,0,0] = [0,0,1]
-  Камера смотрит туда же, куда присоска, но со смещением 89 мм от оси.
-  Присоска в кадр не попадает (край присоски под углом ~40° при VFOV ±32°),
-  объект на оси TCP на дистанции 0.4 м виден со смещением ~12° от центра.
-  Значения — стартовые, уточнить по CAD кронштейна и калибровке (документ 08).
+  TCP z=0.126, радиус присоски ~0.046 м). Кронштейн Camera_Stand_1300: пластина
+  3 мм на фланце (z 0..0.003), лапка с пазами в сторону +X до x=0.0755.
+  Камера прикручена ЗАДНЕЙ панелью к лапке (со стороны присоски) и смотрит
+  вдоль оси инструмента:
+    mount_rpy = 0 -π/2 0  — X камеры (взгляд) -> +Z инструмента, Y (ширина
+                            124 мм) -> +Y (поперёк лапки), Z (верх) -> -X
+                            (верх к оси, нижняя грань с винтом 1/4" — наружу);
+    mount_xyz = 0.075 0 0.015 — нижний винт: нижняя грань на краю лапки
+                            (x=0.075, корпус по высоте 29 мм занимает x
+                            0.046..0.075 — вплотную к присоске, не пересекая);
+                            задняя панель (12 мм позади винта) на пластине
+                            z = 0.015 - 0.012 = 0.003.
+  Присоска частично видна в краю кадра (камера в ~60 мм от оси) — так и на
+  железе. Уточнить по калибровке (документ 08).
 -->
 <robot xmlns:xacro="http://ros.org/wiki/xacro">
   <xacro:macro name="gripper_camera"
       params="camera_model parent:=link_eef name:=gripper_camera
-              mount_xyz:='0.075 0 0.030' mount_rpy:='${pi} ${-pi/2} 0'
+              mount_xyz:='0.075 0 0.015' mount_rpy:='0 ${-pi/2} 0'
               use_nominal_extrinsics:=true add_gz_sensor:=false preview:=false">
-    <!-- Кронштейн: бокс-заглушка (до появления STL из CAD). Привязан к mount_xyz:
-         центр на 18.75 мм (полтолщины бокса) ближе к оси, чем винт камеры;
-         при дефолте 0.075 → x=0.05625, рядом с присоской (до x=0.0375). -->
-    <xacro:property name="_m" value="${[float(v) for v in mount_xyz.split()]}"/>
+    <!-- Кронштейн Camera_Stand_1300 (STL из CAD, мм -> scale 0.001): пластина 3 мм
+         между фланцем и присоской. Диск Ø75 (отверстие Ø30, крепёж) — на фланец
+         соосно link_eef; лапка 45x60 мм с пазами под камеру — в сторону +X
+         link_eef (до x=75.5 мм). Оси меша: Y — толщина (0..3 мм), X — к лапке,
+         Z — поперёк; rpy = (π/2, 0, 0): Y меша -> Z инструмента, Z меша -> -Y. -->
     <joint name="${name}_bracket_joint" type="fixed">
-      <origin xyz="${_m[0] - 0.01875} ${_m[1]} ${_m[2]}" rpy="0 0 0"/>
+      <origin xyz="0 0 0" rpy="0 0 0"/>
       <parent link="${parent}"/>
       <child link="${name}_bracket_link"/>
@@ -30,13 +37,23 @@
     <link name="${name}_bracket_link">
       <inertial>
-        <mass value="0.08"/>
-        <inertia ixx="3.0e-5" ixy="0" ixz="0" iyy="3.0e-5" iyz="0" izz="1.0e-5"/>
+        <!-- алюминий 3 мм, ~0.06 кг; центр масс смещён к лапке -->
+        <origin xyz="0.012 0 0.0015" rpy="0 0 0"/>
+        <mass value="0.06"/>
+        <inertia ixx="2.5e-5" ixy="0" ixz="0" iyy="5.0e-5" iyz="0" izz="7.5e-5"/>
       </inertial>
       <visual>
-        <geometry><box size="0.0375 0.04 0.06"/></geometry>
-        <material name="${name}_bracket_mat"><color rgba="0.15 0.15 0.15 1"/></material>
+        <origin xyz="0 0 0" rpy="${pi/2} 0 0"/>
+        <geometry>
+          <mesh filename="file://$(find quasi_camera_description)/meshes/brackets/camera_stand_1300.stl"
+                scale="0.001 0.001 0.001"/>
+        </geometry>
+        <material name="${name}_bracket_mat"><color rgba="0.75 0.75 0.78 1"/></material>
       </visual>
       <collision>
-        <geometry><box size="0.0375 0.04 0.06"/></geometry>
+        <origin xyz="0 0 0" rpy="${pi/2} 0 0"/>
+        <geometry>
+          <mesh filename="file://$(find quasi_camera_description)/meshes/brackets/camera_stand_1300.stl"
+                scale="0.001 0.001 0.001"/>
+        </geometry>
       </collision>
     </link>

File: src/r2_robot/quasi_cart_description/urdf/c2l-v3.urdf.xacro (robot description, xacro)
@@ -2,8 +2,4 @@
 <robot name="quasi_c2l-v3" xmlns:xacro="http://ros.org/wiki/xacro">
   <xacro:property name="cart_version" value="v3" />
-  <!-- Меш корпуса: default — только если не задан раньше
-       (c2l-v3-scaled.urdf.xacro подставляет масштабированный меш c2) -->
-  <xacro:property name="base_mesh" default="base_link_c2l-v3.stl" />
-  <xacro:property name="base_mesh_scale" default="1 1 1" />
   <!-- Крепление руки (cart-arm.xacro), base_link: по CAD (C2R.000.000.000)
        база руки смещена на 250 мм от центра к ручке (-X) и на 129.5 мм
@@ -11,4 +7,9 @@
        z — верх крыши, та же высота, что у c2 -->
   <xacro:property name="arm_mount_xyz" default="-0.25 -0.1295 0.849" />
+  <!-- Передняя камера (cart-front-camera.xacro): ОЦЕНКА — поза c2 (quasi_ros_c1,
+       enable_camera_orbbec), сдвинутая на +0.1 м вперёд: перед корпуса c2l
+       на 0.1 м дальше (x 0.46 против 0.36). Уточнить по CAD c2l. -->
+  <xacro:property name="front_camera_xyz" default="0.409124 0.0 0.839651" />
+  <xacro:property name="front_camera_rpy" default="${-pi} 0.041 0.0" />
   <link name="base_link">
     <inertial>
@@ -21,6 +22,5 @@
       <origin xyz="0 0 0" rpy="0 0 0" />
       <geometry>
-        <mesh filename="file://$(find quasi_cart_description)/meshes/${base_mesh}"
-              scale="${base_mesh_scale}" />
+        <mesh filename="file://$(find quasi_cart_description)/meshes/base_link_c2l-v3.stl" />
       </geometry>
       <material name="">
@@ -31,6 +31,5 @@
       <origin xyz="0 0 0" rpy="0 0 0" />
       <geometry>
-        <mesh filename="file://$(find quasi_cart_description)/meshes/${base_mesh}"
-              scale="${base_mesh_scale}" />
+        <mesh filename="file://$(find quasi_cart_description)/meshes/base_link_c2l-v3.stl" />
       </geometry>
     </collision>

File: src/r2_robot/quasi_cart_description/urdf/cart-arm.xacro (robot description, xacro)
@@ -5,5 +5,5 @@
   тележки quasi_cart (r2_robot).
   Точка крепления базы руки — свойство arm_mount_xyz (в base_link):
-    - модель тележки может задать своё (c2l-v3*: -0.25 -0.1295 0.849, у края);
+    - модель тележки может задать своё (c2l-v3: -0.25 -0.1295 0.849, у края);
     - иначе дефолт ниже — центр крыши c2 (-0.0075 0 0.849), меш
       base_link_c2-v3.stl: z_top = 0.849 м, x[-0.359 .. 0.359], y[-0.235 .. 0.235].
@@ -29,7 +29,27 @@
   <xacro:arg name="camera_model" default="gemini335le"/>
   <xacro:arg name="gripper_camera_preview" default="false"/>
-  <!-- Модель Gazebo, которую присоска может «приварить» (DetachableJoint).
-       Должна совпадать с именем модели в мире (cart_table_offline.world: pick_box). -->
-  <xacro:arg name="vacuum_target_model" default="pick_box"/>
+  <!-- Модели Gazebo, которые присоска может «приварить» (DetachableJoint), через
+       пробел. Имена = имена моделей в мире, у каждой link «link», модели НЕ static.
+       На каждую — свой плагин и топики /vacuum/<модель>/{attach,detach,state}. -->
+  <xacro:arg name="vacuum_targets" default="pick_box"/>
+  <!-- Плагин DetachableJoint на каждую модель из списка (xacro без циклов —
+       рекурсия по списку) -->
+  <xacro:macro name="vacuum_joints" params="targets">
+    <xacro:if value="${len(targets) > 0}">
+      <gazebo>
+        <plugin filename="gz-sim-detachable-joint-system"
+                name="gz::sim::systems::DetachableJoint">
+          <parent_link>link6</parent_link>
+          <child_model>${targets[0]}</child_model>
+          <child_link>link</child_link>
+          <attach_topic>/vacuum/${targets[0]}/attach</attach_topic>
+          <detach_topic>/vacuum/${targets[0]}/detach</detach_topic>
+          <output_topic>/vacuum/${targets[0]}/state</output_topic>
+          <suppress_child_warning>true</suppress_child_warning>
+        </plugin>
+      </gazebo>
+      <xacro:vacuum_joints targets="${targets[1:]}"/>
+    </xacro:if>
+  </xacro:macro>
   <!-- ==================== Фланец крепления на крыше тележки ==================== -->
   <!-- Точка крепления зависит от тележки: файл модели (<robot_model>.urdf.xacro,
@@ -79,5 +99,5 @@
       gripper_camera_preview="$(arg gripper_camera_preview)"
       ros2_control_plugin="$(arg arm_ros2_control_plugin)"
-      ros2_control_params="$(find xarm_controller)/config/xarm6_controllers.yaml"
+      ros2_control_params="$(find quasi_cart_description)/config/xarm6_controllers_sim.yaml"
       load_gazebo_plugin="true"
       attach_to="arm_mount_link"
@@ -89,8 +109,8 @@
       Физической присоски в gz нет, поэтому «вакуум» = жёсткое соединение
       (fixed joint) между звеном руки и объектом:
-        /vacuum/attach (Empty) -> соединение создаётся с ТЕКУЩИМ взаимным
+        /vacuum/<модель>/attach (Empty) -> соединение создаётся с ТЕКУЩИМ взаимным
                                   положением (объект не телепортируется);
-        /vacuum/detach (Empty) -> соединение удаляется, объект падает;
-        /vacuum/state (String) <- "attached" / "detached".
+        /vacuum/<модель>/detach (Empty) -> соединение удаляется, объект падает;
+        /vacuum/<модель>/state (String) <- "attached" / "detached".
       parent_link = link6: в SDF fixed-суставы URDF схлопываются, и присоска
       (xarm_vacuum_gripper_link), link_eef, камера лежат внутри звена link6
@@ -99,15 +119,6 @@
     -->
     <xacro:if value="$(arg use_sim)">
+      <xacro:vacuum_joints targets="${'$(arg vacuum_targets)'.split()}"/>
       <gazebo>
-        <plugin filename="gz-sim-detachable-joint-system"
-                name="gz::sim::systems::DetachableJoint">
-          <parent_link>link6</parent_link>
-          <child_model>$(arg vacuum_target_model)</child_model>
-          <child_link>link</child_link>
-          <attach_topic>/vacuum/attach</attach_topic>
-          <detach_topic>/vacuum/detach</detach_topic>
-          <output_topic>/vacuum/state</output_topic>
-          <suppress_child_warning>true</suppress_child_warning>
-        </plugin>
         <!-- Поза модели робота в мире (10 Гц) — для проверки касания присоской -->
         <plugin filename="gz-sim-pose-publisher-system"

File: src/r2_robot/quasi_cart_description/urdf/cart-sensors.ign.xacro (robot description, xacro)
@@ -59,4 +59,5 @@
       <topic>/model/cart/imu</topic>
       <ignition_frame_id>imu_link</ignition_frame_id>
+      <frame_id>imu_link</frame_id>
       <always_on>true</always_on>
       <visualize>$(arg imu_visual)</visualize>
@@ -113,4 +114,5 @@
       <topic>/model/cart/tof_sensor1/scan</topic>
       <ignition_frame_id>tof1_link</ignition_frame_id>
+      <frame_id>tof1_link</frame_id>
       <update_rate>10</update_rate>
       <visualize>$(arg tof_visual)</visualize>
@@ -150,4 +152,5 @@
       <topic>/model/cart/tof_sensor2/scan</topic>
       <ignition_frame_id>tof2_link</ignition_frame_id>
+      <frame_id>tof2_link</frame_id>
       <update_rate>10</update_rate>
       <visualize>$(arg tof_visual)</visualize>
@@ -187,4 +190,5 @@
       <topic>/model/cart/tof_sensor3/scan</topic>
       <ignition_frame_id>tof3_link</ignition_frame_id>
+      <frame_id>tof3_link</frame_id>
       <update_rate>10</update_rate>
       <visualize>$(arg tof_visual)</visualize>
@@ -224,4 +228,5 @@
       <topic>/model/cart/tof_sensor4/scan</topic>
       <ignition_frame_id>tof4_link</ignition_frame_id>
+      <frame_id>tof4_link</frame_id>
       <update_rate>10</update_rate>
       <visualize>$(arg tof_visual)</visualize>
@@ -261,4 +266,5 @@
       <topic>/model/cart/tof_sensor5/scan</topic>
       <ignition_frame_id>tof5_link</ignition_frame_id>
+      <frame_id>tof5_link</frame_id>
       <update_rate>10</update_rate>
       <visualize>$(arg tof_visual)</visualize>
@@ -298,4 +304,5 @@
       <topic>/model/cart/tof_sensor6/scan</topic>
       <ignition_frame_id>tof6_link</ignition_frame_id>
+      <frame_id>tof6_link</frame_id>
       <update_rate>10</update_rate>
       <visualize>$(arg tof_visual)</visualize>
@@ -335,4 +342,5 @@
       <topic>/model/cart/tof_sensor7/scan</topic>
       <ignition_frame_id>tof7_link</ignition_frame_id>
+      <frame_id>tof7_link</frame_id>
       <update_rate>10</update_rate>
       <visualize>$(arg tof_visual)</visualize>
@@ -372,4 +380,5 @@
       <topic>/model/cart/tof_sensor8/scan</topic>
       <ignition_frame_id>tof8_link</ignition_frame_id>
+      <frame_id>tof8_link</frame_id>
       <update_rate>10</update_rate>
       <visualize>$(arg tof_visual)</visualize>
@@ -408,4 +417,5 @@
       <topic>/model/cart/lidar</topic>
       <ignition_frame_id>lidar_link</ignition_frame_id>
+      <frame_id>lidar_link</frame_id>
       <pose>0 0 0 0 0 0</pose>
       <visualize>$(arg laser_visual)</visualize>
@@ -445,4 +455,5 @@
       <topic>/model/cart/realsense</topic>
       <ignition_frame_id>camera_rgb_camera_frame</ignition_frame_id>
+      <frame_id>camera_rgb_camera_frame</frame_id>
       <always_on>1</always_on>
       <update_rate>15.0</update_rate>

File: src/r2_robot/quasi_cart_description/urdf/cart_with_arm.urdf.xacro (robot description, xacro)
@@ -4,5 +4,5 @@
   + манипулятор xArm6 с вакуумным гриппером и камерой на ЭФ.
   Рука стоит на крыше тележки: joint arm_mount_joint (base_link -> arm_mount_link,
-  xyz = arm_mount_xyz: для c2 центр -0.0075 0 0.849, для c2l-v3* -0.25 -0.1295 0.849),
+  xyz = arm_mount_xyz: для c2 центр -0.0075 0 0.849, для c2l-v3 -0.25 -0.1295 0.849),
   затем world_joint руки (arm_mount_link -> link_base).
   Этот URDF имеет ПРЯМУЮ ссылку на добавленный манипулятор:
@@ -15,5 +15,5 @@
     <!-- ==================== Аргументы ==================== -->
     <xacro:arg name="use_sim" default="false" />
-    <xacro:arg name="robot_model" default="c2l-v3-scaled" />
+    <xacro:arg name="robot_model" default="c2l-v3" />
     <xacro:arg name="simulator" default="ignition" />
     <xacro:arg name="enable_floor_tofs" default="true" />
@@ -24,4 +24,6 @@
     <xacro:arg name="enable_camera_oak" default="false"/>
     <xacro:arg name="enable_camera_orbbec" default="false"/>
+    <!-- Передняя камера Orbbec Gemini 335Le (cart-front-camera.xacro), /front_camera/... -->
+    <xacro:arg name="front_camera" default="true"/>
     <xacro:arg name="enable_pace_battery" default="true"/>
     <!-- Sensors-система gz объявлена в мирах cart_xarm_bringup/worlds/*.world.
@@ -53,4 +55,8 @@
     <xacro:include filename="cart-drive-${drive}.urdf.xacro"/>
     <xacro:include filename="cart-base.urdf.xacro"/>
+    <xacro:if value="$(arg front_camera)">
+        <xacro:include filename="cart-front-camera.xacro"/>
+        <xacro:cart_front_camera add_gz_sensor="$(arg use_sim)"/>
+    </xacro:if>
     <xacro:if value="$(arg use_sim)">
         <xacro:if value="${var_simulator == 'ignition'}">
